File: daugtherboard/FPGA_scope.kicad_pcb (KiCad board)
At the start: 4 copper layers, 25.5 x 73.2 mm, 23 parts, among them J1 Arduino_MKR_Zero_Socket, J2 Conn_02x06_Odd_Even, J3 HDMI_A, U1 OV5640, U2 TLV71315PDBV, U3 TLV71328PDBV

Commit message: start of PC Software
Connections:
- net /CYC1000/D13_RX renamed /CAM_PCLK
- net /CYC1000/D4 renamed /CAM_HSYNC
- net /CYC1000/D6 renamed /CAM_VSYNC
Changed lines of the file:
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@@
 	(net 14 "+3V3")
 	(net 15 "unconnected-(J1-PadAREF)")
-	(net 16 "/CYC1000/D13_RX")
+	(net 16 "/CAM_PCLK")
 	(net 17 "unconnected-(J1-PadVIN)")
 	(net 18 "/RST")
-	(net 19 "/CYC1000/D6")
-	(net 20 "/CYC1000/D4")
+	(net 19 "/CAM_VSYNC")
+	(net 20 "/CAM_HSYNC")
 	(net 21 "/HDMI_D1-")
 	(net 22 "/HDMI_CEC")
@@
 			(layers "F.Cu" "F.Mask" "F.Paste")
 			(roundrect_rratio 0.15)
-			(net 19 "/CYC1000/D6")
+			(net 19 "/CAM_VSYNC")
 			(pinfunction "VSYNC")
 			(pintype "output")
@@
 			(layers "F.Cu" "F.Mask" "F.Paste")
 			(roundrect_rratio 0.15)
-			(net 20 "/CYC1000/D4")
+			(net 20 "/CAM_HSYNC")
 			(pinfunction "HSYNC")
 			(pintype "output")
@@
 			(layers "F.Cu" "F.Mask" "F.Paste")
 			(roundrect_rratio 0.15)
-			(net 16 "/CYC1000/D13_RX")
+			(net 16 "/CAM_PCLK")
 			(pinfunction "PCLK")
 			(pintype "output")
@@
 			)
 		)
-		(property "Datasheet" ""
+		(property "Datasheet" "https://docs.arduino.cc/hardware/mkr-zero"
 			(at 0 0 90)
 			(layer "F.Fab")
@@
 			)
 		)
-		(property "Description" ""
+		(property "Description" "Socket for Arduino MKR Zero"
 			(at 0 0 90)
 			(layer "F.Fab")
@@
 			(layers "*.Cu" "*.Mask")
 			(remove_unused_layers no)
-			(net 20 "/CYC1000/D4")
+			(net 20 "/CAM_HSYNC")
 			(pinfunction "D4")
 			(pintype "bidirectional")
@@
 			(layers "*.Cu" "*.Mask")
 			(remove_unused_layers no)
-			(net 19 "/CYC1000/D6")
+			(net 19 "/CAM_VSYNC")
 			(pinfunction "D6")
 			(pintype "bidirectional")
@@
 			(layers "*.Cu" "*.Mask")
 			(remove_unused_layers no)
-			(net 16 "/CYC1000/D13_RX")
+			(net 16 "/CAM_PCLK")
 			(pinfunction "D13/RX")
 			(pintype "bidirectional")
